File: IO.kicad_sch (KiCad schematic)
At the start: 5 parts, among them CN2 SM06B-GHS-TB, U10 JBL-102014462, U12 SM06B-SRSS-TB, U8 SM04B-GHS-TB

Commit message: mainly added usart 3, uart 4, and I2C3 connections and planning to add a CAN connection
Parts:
- added R15: 5.1K, Resistor_SMD:R_0201_0603Metric, symbol Device:R_Small
- added R16: 5.1k, Resistor_SMD:R_0201_0603Metric, symbol Device:R_Small
- added U13: SM04B-GHS-TB, LCSC:CONN-SMD_4P-P1.25_SM04B-GHS-TB-LF-SN, symbol LCSC:SM04B-GHS-TB
Connections:
- net +3V3: now also CN2.3
- net GND: now also CN2.4, CN2.7, CN2.8, U8.2, U8.5, U8.6, USBC1.1 (EH), USBC1.2 (EH), USBC1.3 (EH), USBC1.4 (EH), USBC1.A1B12 (GND), USBC1.B1A12 (GND), R15.2, R16.2, U13.2, U13.5, U13.6
- net VBUS: now reaches USBC1.A4B9 (VBUS)
- net VBUS: now also USBC1.B4A9 (VBUS)
- net CC1: now reaches USBC1.A5 (CC1)
- net CC1: now also R15.1
- net D+: now reaches USBC1.A6 (DP1)
- net D+: now also USBC1.B6 (DP2)
- net D-: now reaches USBC1.A7 (DN1)
- net D-: now also USBC1.B7 (DN2)
- net CC2: now reaches USBC1.B5 (CC2)
- net CC2: now also R16.1
- net UART4_RX: now reaches U8.3
- net UART4_TX: now reaches U8.4
- net I2C3_SCL: now reaches CN2.1
- net I2C3_SDA: now reaches CN2.2
- new net USART3_RX: U13.3
- new net USART3_TX: U13.4
- no-connect marks 0 -> 6
Other:
- moved on the sheet: CN2, U8, USBC1
