File: IO.kicad_sch (KiCad schematic)
At the start: 8 parts, among them CN2 SM06B-GHS-TB, U10 JBL-102014462, U12 SM06B-SRSS-TB, U13 SM04B-GHS-TB, U8 SM04B-GHS-TB

Commit message: corrections and IO updated
Connections:
- net I2C3_SCL renamed I2C4_SCL
- net I2C3_SDA renamed I2C4_SDA
Other:
- moved on the sheet: R15, R16
Changed lines of the file:
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@@
 	(wire
 		(pts
-			(xy 35.56 80.01) (xy 46.99 80.01)
+			(xy 124.46 80.01) (xy 135.89 80.01)
 		)
 		(stroke
@@
 	(wire
 		(pts
-			(xy 35.56 93.98) (xy 46.99 93.98)
+			(xy 124.46 93.98) (xy 135.89 93.98)
 		)
 		(stroke
@@
 	)
 	(label "CC1"
-		(at 35.56 80.01 180)
+		(at 124.46 80.01 180)
 		(effects
 			(font
@@
 	)
 	(label "CC2"
-		(at 35.56 93.98 180)
+		(at 124.46 93.98 180)
 		(effects
 			(font
@@
 		)
 	)
-	(hierarchical_label "I2C3_SCL"
+	(hierarchical_label "I2C4_SCL"
 		(shape bidirectional)
 		(at 238.76 140.97 180)
@@
 		)
 	)
-	(hierarchical_label "I2C3_SDA"
+	(hierarchical_label "I2C4_SDA"
 		(shape bidirectional)
 		(at 238.76 143.51 180)
@@
 	(symbol
 		(lib_id "Device:R_Small")
-		(at 46.99 96.52 0)
+		(at 135.89 96.52 0)
 		(unit 1)
 		(body_style 1)
@@
 		(fields_autoplaced yes)
 		(property "Reference" "R16"
-			(at 49.53 95.2499 0)
+			(at 138.43 95.2499 0)
 			(show_name no)
 			(do_not_autoplace no)
@@
 		)
 		(property "Value" "5.1k"
-			(at 49.53 97.7899 0)
+			(at 138.43 97.7899 0)
 			(show_name no)
 			(do_not_autoplace no)
@@
 		)
 		(property "Footprint" "Resistor_SMD:R_0201_0603Metric"
-			(at 46.99 96.52 0)
+			(at 135.89 96.52 0)
 			(hide yes)
 			(show_name no)
@@
 		)
 		(property "Datasheet" ""
-			(at 46.99 96.52 0)
+			(at 135.89 96.52 0)
 			(hide yes)
 			(show_name no)
@@
 		)
 		(property "Description" "Resistor, small symbol"
-			(at 46.99 96.52 0)
+			(at 135.89 96.52 0)
 			(hide yes)
 			(show_name no)
@@
 		)
 		(property "LCSC_PN" ""
-			(at 46.99 96.52 0)
+			(at 135.89 96.52 0)
 			(hide yes)
 			(show_name no)
@@
 	(symbol
 		(lib_id "power:GND")
-		(at 46.99 99.06 0)
+		(at 135.89 99.06 0)
 		(unit 1)
 		(body_style 1)
@@
 		(fields_autoplaced yes)
 		(property "Reference" "#PWR092"
-			(at 46.99 105.41 0)
+			(at 135.89 105.41 0)
 			(hide yes)
 			(show_name no)
@@
 		)
 		(property "Value" "GND"
-			(at 46.99 104.14 0)
+			(at 135.89 104.14 0)
 			(show_name no)
 			(do_not_autoplace no)
@@
 		)
 		(property "Footprint" ""
-			(at 46.99 99.06 0)
+			(at 135.89 99.06 0)
 			(hide yes)
 			(show_name no)
@@
 		)
 		(property "Datasheet" ""
-			(at 46.99 99.06 0)
+			(at 135.89 99.06 0)
 			(hide yes)
 			(show_name no)
@@
 		)
 		(property "Description" "Power symbol creates a global label with name \"GND\" , ground"
-			(at 46.99 99.06 0)
+			(at 135.89 99.06 0)
 			(hide yes)
 			(show_name no)
@@
 	(symbol
 		(lib_id "Device:R_Small")
-		(at 46.99 82.55 0)
+		(at 135.89 82.55 0)
 		(unit 1)
 		(body_style 1)
@@
 		(fields_autoplaced yes)
 		(property "Reference" "R15"
-			(at 49.53 81.2799 0)
+			(at 138.43 81.2799 0)
 			(show_name no)
 			(do_not_autoplace no)
@@
 		)
 		(property "Value" "5.1K"
-			(at 49.53 83.8199 0)
+			(at 138.43 83.8199 0)
 			(show_name no)
 			(do_not_autoplace no)
@@
 		)
 		(property "Footprint" "Resistor_SMD:R_0201_0603Metric"
-			(at 46.99 82.55 0)
+			(at 135.89 82.55 0)
 			(hide yes)
 			(show_name no)
@@
 		)
 		(property "Datasheet" ""
-			(at 46.99 82.55 0)
+			(at 135.89 82.55 0)
 			(hide yes)
 			(show_name no)
@@
 		)
 		(property "Description" "Resistor, small symbol"
-			(at 46.99 82.55 0)
+			(at 135.89 82.55 0)
 			(hide yes)
 			(show_name no)
@@
 		)
 		(property "LCSC_PN" ""
-			(at 46.99 82.55 0)
+			(at 135.89 82.55 0)
 			(hide yes)
 			(show_name no)
@@
 	(symbol
 		(lib_id "power:GND")
-		(at 46.99 85.09 0)
+		(at 135.89 85.09 0)
 		(unit 1)
 		(body_style 1)
@@
 		(dnp no)
 		(property "Reference" "#PWR091"
-			(at 46.99 91.44 0)
+			(at 135.89 91.44 0)
 			(hide yes)
 			(show_name no)
@@
 		)
 		(property "Value" "GND"
-			(at 46.99 90.17 0)
+			(at 135.89 90.17 0)
 			(show_name no)
 			(do_not_autoplace no)
@@
 		)
 		(property "Footprint" ""
-			(at 46.99 85.09 0)
+			(at 135.89 85.09 0)
 			(hide yes)
 			(show_name no)
@@
 		)
 		(property "Datasheet" ""
-			(at 46.99 85.09 0)
+			(at 135.89 85.09 0)
 			(hide yes)
 			(show_name no)
@@
 		)
 		(property "Description" "Power symbol creates a global label with name \"GND\" , ground"
-			(at 46.99 85.09 0)
-			(hide yes)
-			(show_name no)
+			(at 135.89 85.09 0)
+			(hide yes)
+			(show_name no)

Commit message: added in RF componentys and updated and reviewed STM connections
Parts:
- added C37, C43, C47, C48: 1uF, Capacitor_SMD:C_0201_0603Metric_Pad0.64x0.40mm_HandSolder, symbol Device:C_Small
- added C46: 100uF, Capacitor_SMD:C_0201_0603Metric_Pad0.64x0.40mm_HandSolder, symbol Device:C_Small
- added CN3: SM07B-SRSS-TB, LCSC:CONN-SMD_SM07B-SRSS-TB, symbol LCSC:SM07B-SRSS-TB
- added D2: USBLC6-2SC6, LCSC:SOT-23-6_L2.9-W1.6-P0.95-LS2.8-BL, symbol LCSC:USBLC6-2SC6
- added R19: 300k, Resistor_SMD:R_0201_0603Metric, symbol Device:R_Small
- added R20: 100k, Resistor_SMD:R_0201_0603Metric, symbol Device:R_Small
- added U6: TPS2116DRLR, LCSC:SOT-583-8_L2.1-W1.6-P0.50-LS1.6-BL, symbol LCSC:TPS2116DRLR
Connections:
- net D+: now also D2.3, D2.4
- net D-: now also D2.1, D2.6
- net GND: now also C37.2, C43.2, C46.2, C47.2, C48.2, CN3.7, D2.2, R20.1, U6.1 (GND)
- net VBUS: now also C48.1, D2.5, U6.6 (VIN2)
- new net 5V: C43.1, C46.1, U6.2 (VOUT), U6.7 (VOUT)
- new net 5V_BUCK: C37.1, C47.1, R19.2, U6.3 (VIN1), U6.5 (MODE)
- new net DSHOT_M1: CN3.3
- new net DSHOT_M2: CN3.4
- new net DSHOT_M3: CN3.5
- new net DSHOT_M4: CN3.6
- new net KISS_TELEM: CN3.2
- new net PR: R19.1, R20.2, U6.4 (PR1)
- new net VBAT: CN3.1
Other:
- moved on the sheet: R15, R16
